Commit message: Fix unsupported value in vs068.urdf

File: denso_robot_descriptions/vs068_description/vs068.urdf (robot description, URDF)
Before this commit: robot vs068, 7 links, 6 joints
Joints:
- joint joint_5: origin xyz=0.000000 0.000000 ${0.340-0.197} rpy=0.000000 0.000000 0.000000 -> xyz=0.000000 0.000000 0.143 rpy=0.000000 0.000000 0.000000

Commit message: Change joint limits for wrobot

File: denso_robot_descriptions/vs068_description/vs068.urdf (robot description, URDF)
Before this commit: robot vs068, 7 links, 6 joints
Joints:
- joint joint_1: limit lower=-2.96706 upper=2.96706 effort=1 velocity=3.92699081698724 -> lower=-2.9670597283903604 upper=2.9670597283903604 effort=1 velocity=3.92699081698724
- joint joint_2: limit lower=-2.094395 upper=2.094395 effort=1 velocity=2.61799387799149 -> lower=0.0 upper=2.356194490192345 effort=1 velocity=2.61799387799149
- joint joint_3: limit lower=-2.181662 upper=2.70526 effort=1 velocity=2.85832571599111 -> lower=0.0 upper=2.670353755551324 effort=1 velocity=2.85832571599111
- joint joint_4: limit lower=-4.712389 upper=4.712389 effort=1 velocity=3.92699081698724 -> lower=-2.792526803190927 upper=2.792526803190927 effort=1 velocity=3.92699081698724
- joint joint_6: limit lower=-6.283185 upper=6.283185 effort=1 velocity=6.28318530717959 -> lower=-4.1887902047863905 upper=4.1887902047863905 effort=1 velocity=6.28318530717959

File: denso_robot_descriptions/vs068_description/vs068.xacro (robot description, xacro)
@@ -54,5 +54,5 @@
       <origin rpy="0.000000 0.000000 0.000000" xyz="0.000000 0.000000 0.1975" />
       <axis xyz="0.000000 0.000000 1.000000" />
-      <limit effort="1" lower="-2.96706" upper="2.96706" velocity="3.92699081698724" />
+      <limit effort="1" lower="-2.8797932657906435" upper="2.8797932657906435" velocity="3.92699081698724" />
       <dynamics damping="0" friction="0" />
     </joint>
@@ -92,5 +92,5 @@
       <origin rpy="0.000000 0.000000 0.000000" xyz="0.030 0.000 0.1975" />
       <axis xyz="0.000000 1.000000 0.000000" />
-      <limit effort="1" lower="-2.094395" upper="2.094395" velocity="2.61799387799149" />
+      <limit effort="1" lower="0.0" upper="2.2689280275926285" velocity="2.61799387799149" />
       <dynamics damping="0" friction="0" />
     </joint>
@@ -130,5 +130,5 @@
       <origin rpy="0.000000 0.000000 0.000000" xyz="0.000000 0.000000 0.340" />
       <axis xyz="0.000000 1.000000 0.000000" />
-      <limit effort="1" lower="-2.70526" upper="2.70526" velocity="2.85832571599111" />
+      <limit effort="1" lower="0.6981317007977318" upper="2.356194490192345" velocity="2.85832571599111" />
       <dynamics damping="0" friction="0" />
     </joint>
@@ -168,5 +168,5 @@
       <origin rpy="0.000000 0.000000 0.000000" xyz="-0.020 0.000 0.197" />
       <axis xyz="0.000000 0.000000 1.000000" />
-      <limit effort="1" lower="-1.57" upper="1.57" velocity="3.92699081698724" />
+      <limit effort="1" lower="-2.705260340591211" upper="2.705260340591211" velocity="3.92699081698724" />
       <dynamics damping="0" friction="0" />
     </joint>
@@ -206,5 +206,5 @@
       <origin rpy="0.000000 0.000000 0.000000" xyz="0.000000 0.000000 0.143" />
       <axis xyz="-0.000000 1.000000 -0.000000" />
-      <limit effort="1" lower="-2.094395" upper="2.094395" velocity="3.02168853397778" />
+      <limit effort="1" lower="-2.007128639793479" upper="2.007128639793479" velocity="3.02168853397778" />
       <dynamics damping="0" friction="0" />
     </joint>
@@ -231,5 +231,5 @@
       <origin rpy="0.000000 0.000000 0.000000" xyz="0.000000 0.000000 0.115" />
       <axis xyz="-0.000000 -0.000000 1.000000" />
-      <limit effort="1" lower="-6.283185" upper="6.283185" velocity="6.28318530717959" />
+      <limit effort="1" lower="-4.101523742186674" upper="4.101523742186674" velocity="6.28318530717959" />
       <dynamics damping="0" friction="0" />
     </joint>
